File: 202011a/kicad/md202011a.kicad_pcb (KiCad board)
At the start: 2 copper layers, 79 x 59.5 mm, 47 parts, among them J101 MCU, J102 SocketA, J103 SocketB, J104 LED_EN, J201 PB, J202 PWR, Q101 MMBT3904, SW301 Y, SW302 O, SW303 R, SW304 G, SW305 RESET, U101 STC15W104, U201 LM358, U301 ATtiny13A-PU

Commit message: Correct the probe resistor value to 2.2K
Parts:
- R208: value 470 -> 2.2K
