File: 202101a/kicad/202101a.kicad_pcb (KiCad board)
At the start: 2 copper layers, 68.8 x 53.6 mm, 49 parts, among them J1 Barrel_Jack_Switch, J2 USB_B, J3 ICSP, J4 ExtIO, Q1 DMG2301L, SW1 RESET, U1 AMS1117-5.0, U2 XC6206P332MR, U3 LM358, U4 CH340G, U5 ATmega328-PU, U6 ATmega328-AU, Y1 12MHz, Y2 16MHz

Commit message: Add some labels on the B.SilkS layer.
And update the settings of the pages.
Other:
- board text added: "0 RX"
- board text added: "1 TX"
- board text added: "10~~"
- board text added: "11~~"
- board text added: "3~~."
- board text added: "5~~."
- board text added: "6~~."
- board text added: "9~~"
