File: 202106a-mrx40/kicad/202106a-mrx40.kicad_pcb (KiCad board)
At the start: 2 copper layers, 80 x 40 mm, 37 parts, among them J1 Ant, J2 Mute, J3 USB_B_Micro, J4 5V, J5 AF, U1 NE602, U2 FM8002A, Y1 7.023

Commit message: Fix BB910 pin error
Parts:
- D1: footprint Package_TO_SOT_THT:TO-92-2 -> bg1ren:TO-92-2-21
- moved D1 2.50 mm to (114.0, 166.5), turned to 90 degrees
Other:
- board text added: "MRX-40 MOD by BG1REN - 20210629 v2"
- board text removed: "MRX-40 MOD by BG1REN - 20210628 v1"
